File: PCB_Laserdinges/Laserdinges.kicad_pcb (KiCad board)
At the start: 2 copper layers, 63.1 x 49.9 mm, 30 parts, among them J1 Conn_01x04_Pin, J2 Barrel_Jack, SW1 SW_Push, SW2 SW_Push, SW3 SW_SPST, SW4 SW_DIP_x01, SW5 SW_DIP_x01, SW6 SW_DIP_x01, U1 ESP32-WROOM-32, U2 AMS1117-3.3, U4 MP1584

Commit message: pcb_v2
Parts:
- J1: footprint Connector_PinHeader_2.00mm:PinHeader_1x04_P2.00mm_Vertical -> Connector_PinHeader_2.54mm:PinHeader_1x04_P2.54mm_Vertical
- SW3, SW4, SW5, SW6, U5: footprint Connector_PinHeader_2.00mm:PinHeader_1x02_P2.00mm_Vertical -> Connector_PinHeader_2.54mm:PinHeader_1x02_P2.54mm_Vertical
- U3: footprint Connector_PinHeader_2.00mm:PinHeader_1x05_P2.00mm_Vertical -> Connector_PinHeader_2.54mm:PinHeader_1x05_P2.54mm_Vertical
- moved U3 2.74 mm to (132.3, 91.9)
- moved J1 0.75 mm to (132.8, 76.5)
- moved SW6 0.43 mm to (119.1, 98.6)
- moved SW5 0.39 mm to (114.6, 98.6)
- moved SW3 0.33 mm to (105.9, 100.8)
- moved U1 0.11 mm to (113.9, 72.9)
Routing:
- net A4: track 63.7 -> 72.9 mm
- net VDD: track 81.7 -> 85.8 mm
- net Net-(U3-VRX): track 17.0 -> 15.6 mm
- net TX0: track 13.9 -> 12.7 mm
- net GPIO19: track 33.4 -> 34.6 mm
- net RX0: track 13.0 -> 12.0 mm
- net +3.3V: track 137.7 -> 138.6 mm
- net Net-(U3-VRY): track 6.32 -> 5.43 mm
- net GND: vias 23 -> 27
Other:
- board size 63.1 x 49.9 mm -> 60.6 x 49.9 mm
- board text added: "o"
- board text added: "|"
