File: PCB_Motordinges/Motordinges/Motordinges.kicad_pcb (KiCad board)
At the start: 2 copper layers, 65.6 x 42.9 mm, 22 parts, among them J1 Conn_01x04_Pin, J2 Barrel_Jack, SW1 EN, SW2 FLASH, U1 ESP32-WROOM-32, U2 MP1584, U3 AMS1117-3.3

Commit message: pcb_v2
Parts:
- removed the Motor1 at (140.6, 66.8)
- removed the Motor2 at (133.2, 67.0)
- added Motor1: Conn_01x02_Pin, Connector_PinHeader_2.54mm:PinHeader_1x02_P2.54mm_Vertical, F.Cu at (140.5, 67.1)
- added Motor1: Conn_01x02_Pin, TerminalBlock:TerminalBlock_bornier-2_P5.08mm, F.Cu at (122.4, 74.2)
- added Motor2: Conn_01x02_Pin, TerminalBlock:TerminalBlock_bornier-2_P5.08mm, F.Cu at (111.8, 74.2)
- added Motor2: Conn_01x02_Pin, Connector_PinHeader_2.54mm:PinHeader_1x02_P2.54mm_Vertical, F.Cu at (133.9, 67.1)
- J1: footprint Connector_PinHeader_2.00mm:PinHeader_1x04_P2.00mm_Vertical -> Connector_PinHeader_2.54mm:PinHeader_1x04_P2.54mm_Vertical
- moved SW2 4.92 mm to (130.0, 65.0)
- moved R2 3.30 mm to (131.1, 57.7)
- moved SW1 3.08 mm to (106.9, 68.3)
- moved R6 2.31 mm to (131.3, 53.6)
- moved J1 1.58 mm to (138.4, 57.9)
- moved R5 1.49 mm to (131.8, 47.2)
Routing:
- net +3.3V: track 148.6 -> 141.8 mm
- net Net-(J5-Pin_2): track 75.2 -> 78.5 mm
- net /EN: track 21.3 -> 19.3 mm
- net RX0: track 16.0 -> 14.1 mm
- net GPIO13: track 28.0 -> 29.2 mm
- net TX0: track 15.6 -> 14.4 mm
- net GPIO5: track 3.51 -> 4.54 mm
- net A8: track 38.1 -> 37.1 mm
- net GPIO23: track 39.5 -> 40.2 mm
- net GPIO0: track 7.20 -> 6.64 mm
Other:
- outline, holes or cut-outs redrawn
- board text added: "+12V"
- board text added: "Sien Peerlinck, Thibaut Dalez Motordinges v2"
- board text removed: "12V"
- board text removed: "Sien Peerlinck, Thibaut Dalez Motordinges v1"
